Commit message: Add wheel links and joints to my_robot

File: urdf/my_robot.xacro (robot description, xacro)
@@ -1,3 +1,3 @@
-<?xml version='1.0'?>
+<?xml version="1.0"?>
 <robot name="my_robot" xmlns:xacro="http://www.ros.org/wiki/xacro">
     <link name="robot_footprint"/>
@@ -7,5 +7,5 @@
         <child link="chassis" />
     </joint>
-    <link name='chassis'>
+    <link name="chassis">
         <pose>0 0 0.1 0 0 0</pose>
         <inertial>
@@ -18,5 +18,5 @@
             />
         </inertial>
-        <collision name='collision'>
+        <collision name="collision">
             <origin xyz="0 0 0" rpy=" 0 0 0"/>
             <geometry>
@@ -24,5 +24,5 @@
             </geometry>
         </collision>
-        <visual name='chassis_visual'>
+        <visual name="chassis_visual">
             <origin xyz="0 0 0" rpy=" 0 0 0"/>
             <geometry>
@@ -30,5 +30,5 @@
             </geometry>
         </visual>
-        <collision name='back_caster_collision'>
+        <collision name="back_caster_collision">
             <origin xyz="-0.15 0 -0.05" rpy=" 0 0 0"/>
             <geometry>
@@ -36,5 +36,5 @@
             </geometry>
         </collision>
-        <visual name='back_caster_visual'>
+        <visual name="back_caster_visual">
             <origin xyz="-0.15 0 -0.05" rpy=" 0 0 0"/>
             <geometry>
@@ -42,5 +42,5 @@
             </geometry>
         </visual>
-        <collision name='front_caster_collision'>
+        <collision name="front_caster_collision">
             <origin xyz="0.15 0 -0.05" rpy=" 0 0 0"/>
             <geometry>
@@ -48,5 +48,5 @@
             </geometry>
         </collision>
-        <visual name='front_caster_visual'>
+        <visual name="front_caster_visual">
             <origin xyz="0.15 0 -0.05" rpy=" 0 0 0"/>
             <geometry>
@@ -55,3 +55,63 @@
         </visual>
     </link>
+    <link name="left_wheel">
+        <visual name="left_wheel_visual">
+            <origin xyz="0 0 0" rpy="0 1.5707 1.5707"/>
+            <geometry>
+                <cylinder radius="0.1" length="0.05"/>
+            </geometry>
+        </visual>
+        <collision name="left_wheel_collision">
+            <origin xyz="0 0 0" rpy="0 1.5707 1.5707"/>
+            <geometry>
+                <cylinder radius="0.1" length="0.05"/>
+            </geometry>
+        </collision>
+        <inertial>
+            <origin xyz="0 0 0" rpy="0 1.5707 1.5707"/>
+            <mass value="5.0"/>
+            <inertia
+                    ixx="0.1" ixy="0" ixz="0"
+                    iyy="0.1" iyz="0"
+                    izz="0.1"/>
+        </inertial>
+    </link>
+    <link name="right_wheel">
+        <visual name="right_wheel_visual">
+            <origin xyz="0 0 0" rpy="0 1.5707 1.5707"/>
+            <geometry>
+                <cylinder radius="0.1" length="0.05"/>
+            </geometry>
+        </visual>
+        <collision name="right_wheel_collision">
+            <origin xyz="0 0 0" rpy="0 1.5707 1.5707"/>
+            <geometry>
+                <cylinder radius="0.1" length="0.05"/>
+            </geometry>
+        </collision>
+        <inertial>
+            <origin xyz="0 0 0" rpy="0 1.5707 1.5707"/>
+            <mass value="5.0"/>
+            <inertia
+                    ixx="0.1" ixy="0" ixz="0"
+                    iyy="0.1" iyz="0"
+                    izz="0.1"/>
+        </inertial>
+    </link>
+    <joint type="continuous" name="left_wheel_hinge">
+        <origin xyz="0 0.15 0" rpy="0 0 0"/>
+        <child link="left_wheel"/>
+        <parent link="chassis"/>
+        <axis xyz="0 1 0" rpy="0 0 0"/>
+        <limit effort="10000" velocity="1000"/>
+        <dynamics damping="1.0" friction="1.0"/>
+    </joint>
+    <joint type="continuous" name="right_wheel_hinge">
+        <origin xyz="0 -0.15 0" rpy="0 0 0"/>
+        <child link="right_wheel"/>
+        <parent link="chassis"/>
+        <axis xyz="0 1 0" rpy="0 0 0"/>
+        <limit effort="10000" velocity="1000"/>
+        <dynamics damping="1.0" friction="1.0"/>
+    </joint>
 </robot>

Commit message: Add camera link / joint

File: urdf/my_robot.xacro (robot description, xacro)
@@ -115,3 +115,34 @@
         <dynamics damping="1.0" friction="1.0"/>
     </joint>
+    <link name="camera">
+        <visual>
+            <origin xyz="0 0 0" rpy="0 0 0"/>
+            <geometry>
+                <box size="0.05 0.05 0.05"/>
+            </geometry>
+        </visual>
+        <collision>
+            <origin xyz="0 0 0" rpy="0 0 0"/>
+            <geometry>
+                <box size="0.05 0.05 0.05"/>
+            </geometry>
+        </collision>
+        <inertial>
+            <mass value="0.1"/>
+            <origin xyz="0.0 0 0" rpy=" 0 0 0"/>
+            <box_inertia
+                    m="0.1" x="0.05" y="0.05" z="0.05"/>
+            <inertia
+                    ixx="1e-6" ixy="0" ixz="0"
+                    iyy="1e-6" iyz="0"
+                    izz="1e-6"
+            />
+        </inertial>
+    </link>
+    <joint type="fixed" name="camera_joint">
+        <axis xyz="0 1 0" rpy="0 0 0"/>
+        <origin xyz="0.2 0 0" rpy="0 0 0"/>
+        <child link="camera"/>
+        <parent link="chassis"/>
+    </joint>
 </robot>

Commit message: Add LiDAR sensor using Hokuyo Collada mesh

File: urdf/my_robot.xacro (robot description, xacro)
@@ -143,6 +143,35 @@
         <axis xyz="0 1 0" rpy="0 0 0"/>
         <origin xyz="0.2 0 0" rpy="0 0 0"/>
+        <parent link="chassis"/>
         <child link="camera"/>
+    </joint>
+    <link name="hokuyo">
+        <visual>
+            <origin xyz="0 0 0" rpy="0 0 0"/>
+            <geometry>
+                <mesh filename="package://my_robot/meshes/hokuyo.dae" />
+            </geometry>
+        </visual>
+        <collision>
+            <origin xyz="0 0 0" rpy="0 0 0"/>
+            <geometry>
+                <box size="0.1 0.1 0.1"/>
+            </geometry>
+        </collision>
+        <inertial>
+            <mass value="1e-5"/>
+            <origin xyz="0.0 0 0" rpy=" 0 0 0"/>
+            <inertia
+                    ixx="1e-6" ixy="0" ixz="0"
+                    iyy="1e-6" iyz="0"
+                    izz="1e-6"
+            />
+        </inertial>
+    </link>
+    <joint type="fixed" name="hokuyo_joint">
+        <axis xyz="0 1 0" rpy="0 0 0"/>
+        <origin xyz="0.15 0 0.1" rpy="0 0 0"/>
         <parent link="chassis"/>
+        <child link="hokuyo"/>
     </joint>
 </robot>

Commit message: Add horrible gazebo/material to wheels

File: urdf/my_robot.xacro (robot description, xacro)
@@ -77,4 +77,7 @@
         </inertial>
     </link>
+    <gazebo reference="left_wheel">
+        <material>Gazebo/Green</material>
+    </gazebo>
     <link name="right_wheel">
         <visual name="right_wheel_visual">
@@ -99,4 +102,7 @@
         </inertial>
     </link>
+    <gazebo reference="right_wheel">
+        <material>Gazebo/Green</material>
+    </gazebo>
     <joint type="continuous" name="left_wheel_hinge">
         <origin xyz="0 0.15 0" rpy="0 0 0"/>

Commit message: Update my_robot

File: urdf/my_robot.xacro (robot description, xacro)
@@ -32,27 +32,41 @@
         </visual>
         <collision name="back_caster_collision">
-            <origin xyz="-0.15 0 -0.05" rpy=" 0 0 0"/>
+            <origin xyz="-0.15 0 -0.06" rpy="0 0 0"/>
             <geometry>
-                <sphere radius="0.0499"/>
+                <sphere radius="0.04"/>
             </geometry>
         </collision>
         <visual name="back_caster_visual">
-            <origin xyz="-0.15 0 -0.05" rpy=" 0 0 0"/>
+            <origin xyz="-0.15 0 -0.06" rpy="0 0 0"/>
             <geometry>
-                <sphere radius="0.05"/>
+                <sphere radius="0.04"/>
             </geometry>
         </visual>
-        <collision name="front_caster_collision">
-            <origin xyz="0.15 0 -0.05" rpy=" 0 0 0"/>
+        <!--
+        <collision name="back_left_caster_collision">
+            <origin xyz="-0.15 0.05 -0.06" rpy="0 0 0"/>
             <geometry>
-                <sphere radius="0.0499"/>
+                <sphere radius="0.04"/>
             </geometry>
         </collision>
-        <visual name="front_caster_visual">
-            <origin xyz="0.15 0 -0.05" rpy=" 0 0 0"/>
+        <visual name="back_left_caster_visual">
+            <origin xyz="-0.15 0.05 -0.06" rpy="0 0 0"/>
             <geometry>
-                <sphere radius="0.05"/>
+                <sphere radius="0.04"/>
             </geometry>
         </visual>
+        <collision name="back_right_caster_collision">
+            <origin xyz="-0.15 -0.05 -0.06" rpy="0 0 0"/>
+            <geometry>
+                <sphere radius="0.04"/>
+            </geometry>
+        </collision>
+        <visual name="back_right_caster_visual">
+            <origin xyz="-0.15 -0.05 -0.06" rpy="0 0 0"/>
+            <geometry>
+                <sphere radius="0.04"/>
+            </geometry>
+        </visual>
+        -->
     </link>
     <link name="left_wheel">
@@ -60,5 +74,5 @@
             <origin xyz="0 0 0" rpy="0 1.5707 1.5707"/>
             <geometry>
-                <cylinder radius="0.1" length="0.05"/>
+                <cylinder radius="0.075" length="0.05"/>
             </geometry>
         </visual>
@@ -66,5 +80,5 @@
             <origin xyz="0 0 0" rpy="0 1.5707 1.5707"/>
             <geometry>
-                <cylinder radius="0.1" length="0.05"/>
+                <cylinder radius="0.075" length="0.05"/>
             </geometry>
         </collision>
@@ -78,12 +92,9 @@
         </inertial>
     </link>
-    <gazebo reference="left_wheel">
-        <material>Gazebo/Green</material>
-    </gazebo>
     <link name="right_wheel">
         <visual name="right_wheel_visual">
             <origin xyz="0 0 0" rpy="0 1.5707 1.5707"/>
             <geometry>
-                <cylinder radius="0.1" length="0.05"/>
+                <cylinder radius="0.075" length="0.05"/>
             </geometry>
         </visual>
@@ -91,5 +102,5 @@
             <origin xyz="0 0 0" rpy="0 1.5707 1.5707"/>
             <geometry>
-                <cylinder radius="0.1" length="0.05"/>
+                <cylinder radius="0.075" length="0.05"/>
             </geometry>
         </collision>
@@ -103,9 +114,6 @@
         </inertial>
     </link>
-    <gazebo reference="right_wheel">
-        <material>Gazebo/Green</material>
-    </gazebo>
     <joint type="continuous" name="left_wheel_hinge">
-        <origin xyz="0 0.15 0" rpy="0 0 0"/>
+        <origin xyz="0.1 0.13 -0.025" rpy="0 0 0"/>
         <child link="left_wheel"/>
         <parent link="chassis"/>
@@ -115,5 +123,5 @@
     </joint>
     <joint type="continuous" name="right_wheel_hinge">
-        <origin xyz="0 -0.15 0" rpy="0 0 0"/>
+        <origin xyz="0.1 -0.13 -0.025" rpy="0 0 0"/>
         <child link="right_wheel"/>
         <parent link="chassis"/>
@@ -178,7 +186,13 @@
     <joint type="fixed" name="hokuyo_joint">
         <axis xyz="0 1 0" rpy="0 0 0"/>
-        <origin xyz="0.15 0 0.1" rpy="0 0 0"/>
+        <origin xyz="0.15 0 0.05" rpy="0 0 0"/>
         <parent link="chassis"/>
         <child link="hokuyo"/>
     </joint>
+    <gazebo reference="right_wheel">
+        <material>Gazebo/DarkGrey</material>
+    </gazebo>
+    <gazebo reference="left_wheel">
+        <material>Gazebo/DarkGrey</material>
+    </gazebo>
 </robot>

Commit message: Remove unused caster wheels

File: urdf/my_robot.xacro (robot description, xacro)
@@ -43,30 +43,4 @@
             </geometry>
         </visual>
-        <!--
-        <collision name="back_left_caster_collision">
-            <origin xyz="-0.15 0.05 -0.06" rpy="0 0 0"/>
-            <geometry>
-                <sphere radius="0.04"/>
-            </geometry>
-        </collision>
-        <visual name="back_left_caster_visual">
-            <origin xyz="-0.15 0.05 -0.06" rpy="0 0 0"/>
-            <geometry>
-                <sphere radius="0.04"/>
-            </geometry>
-        </visual>
-        <collision name="back_right_caster_collision">
-            <origin xyz="-0.15 -0.05 -0.06" rpy="0 0 0"/>
-            <geometry>
-                <sphere radius="0.04"/>
-            </geometry>
-        </collision>
-        <visual name="back_right_caster_visual">
-            <origin xyz="-0.15 -0.05 -0.06" rpy="0 0 0"/>
-            <geometry>
-                <sphere radius="0.04"/>
-            </geometry>
-        </visual>
-        -->
     </link>
     <link name="left_wheel">

Commit message: Add funky LED to funkybot

File: urdf/my_robot.xacro (robot description, xacro)
@@ -44,4 +44,18 @@
         </visual>
     </link>
+    <link name="led_visual">
+        <visual>
+            <origin xyz="0 0 0" rpy="0 0 0"/>
+            <geometry>
+                <sphere radius="0.005"/>
+            </geometry>
+        </visual>
+    </link>
+    <joint type="fixed" name="led_visual_hinge">
+        <origin xyz="-0.15 0.05 0.05" rpy=" 0 0 0"/>
+        <child link="led_visual"/>
+        <parent link="chassis"/>
+        <axis xyz="0 0 1" rpy="0 0 0"/>
+    </joint>
     <link name="left_wheel">
         <visual name="left_wheel_visual">
@@ -170,3 +184,6 @@
         <material>Gazebo/DarkGrey</material>
     </gazebo>
+    <gazebo reference="led_visual">
+        <material>Gazebo/GreenGlow</material>
+    </gazebo>
 </robot>

Commit message: Update material

File: urdf/my_robot.xacro (robot description, xacro)
@@ -187,3 +187,9 @@
         <material>Gazebo/GreenGlow</material>
     </gazebo>
+    <gazebo reference="chassis">
+        <material>Gazebo/Gold</material>
+    </gazebo>
+    <gazebo reference="camera">
+        <material>Gazebo/Grey</material>
+    </gazebo>
 </robot>
