Commit message: Change my_robot to where_am_i

File: src/where_am_i/urdf/my_robot.xacro (robot description, xacro)
@@ -1,5 +1,5 @@
 <?xml version="1.0"?>
 <robot name="my_robot" xmlns:xacro="http://www.ros.org/wiki/xacro">
-    <xacro:include filename="$(find my_robot)/urdf/my_robot.gazebo" />
+    <xacro:include filename="$(find where_am_i)/urdf/my_robot.gazebo" />
     <link name="robot_footprint"/>
     <joint name="robot_footprint_joint" type="fixed">
@@ -153,5 +153,5 @@
             <origin xyz="0 0 0" rpy="0 0 0"/>
             <geometry>
-                <mesh filename="package://my_robot/meshes/hokuyo.dae" />
+                <mesh filename="package://where_am_i/meshes/hokuyo.dae" />
             </geometry>
         </visual>

Commit message: Separate wheels and increase torque

File: src/where_am_i/urdf/my_robot.xacro (robot description, xacro)
@@ -103,5 +103,5 @@
     </link>
     <joint type="continuous" name="left_wheel_hinge">
-        <origin xyz="0.1 0.13 -0.025" rpy="0 0 0"/>
+        <origin xyz="0.1 0.15 -0.025" rpy="0 0 0"/>
         <child link="left_wheel"/>
         <parent link="chassis"/>
@@ -111,5 +111,5 @@
     </joint>
     <joint type="continuous" name="right_wheel_hinge">
-        <origin xyz="0.1 -0.13 -0.025" rpy="0 0 0"/>
+        <origin xyz="0.1 -0.15 -0.025" rpy="0 0 0"/>
         <child link="right_wheel"/>
         <parent link="chassis"/>

Commit message: Update bot center of mass

File: src/where_am_i/urdf/my_robot.xacro (robot description, xacro)
@@ -12,5 +12,5 @@
         <inertial>
             <mass value="15.0"/>
-            <origin xyz="0.0 0 0" rpy=" 0 0 0"/>
+            <origin xyz="-0.05 0 -0.05" rpy="0 0 0"/>
             <inertia
                     ixx="0.1" ixy="0" ixz="0"

Commit message: Change to skid steer drive

File: src/where_am_i/urdf/my_robot.xacro (robot description, xacro)
@@ -12,5 +12,5 @@
         <inertial>
             <mass value="15.0"/>
-            <origin xyz="-0.05 0 -0.05" rpy="0 0 0"/>
+            <origin xyz="0 0 0" rpy="0 0 0"/>
             <inertia
                     ixx="0.1" ixy="0" ixz="0"
@@ -29,16 +29,4 @@
             <geometry>
                 <box size=".4 .2 .1"/>
-            </geometry>
-        </visual>
-        <collision name="back_caster_collision">
-            <origin xyz="-0.15 0 -0.06" rpy="0 0 0"/>
-            <geometry>
-                <sphere radius="0.04"/>
-            </geometry>
-        </collision>
-        <visual name="back_caster_visual">
-            <origin xyz="-0.15 0 -0.06" rpy="0 0 0"/>
-            <geometry>
-                <sphere radius="0.04"/>
             </geometry>
         </visual>
@@ -58,59 +46,119 @@
         <axis xyz="0 0 1" rpy="0 0 0"/>
     </joint>
-    <link name="left_wheel">
-        <visual name="left_wheel_visual">
-            <origin xyz="0 0 0" rpy="0 1.5707 1.5707"/>
-            <geometry>
-                <cylinder radius="0.075" length="0.05"/>
-            </geometry>
-        </visual>
-        <collision name="left_wheel_collision">
-            <origin xyz="0 0 0" rpy="0 1.5707 1.5707"/>
-            <geometry>
-                <cylinder radius="0.075" length="0.05"/>
-            </geometry>
-        </collision>
-        <inertial>
-            <origin xyz="0 0 0" rpy="0 1.5707 1.5707"/>
-            <mass value="5.0"/>
-            <inertia
-                    ixx="0.1" ixy="0" ixz="0"
-                    iyy="0.1" iyz="0"
-                    izz="0.1"/>
-        </inertial>
-    </link>
-    <link name="right_wheel">
-        <visual name="right_wheel_visual">
-            <origin xyz="0 0 0" rpy="0 1.5707 1.5707"/>
-            <geometry>
-                <cylinder radius="0.075" length="0.05"/>
-            </geometry>
-        </visual>
-        <collision name="right_wheel_collision">
-            <origin xyz="0 0 0" rpy="0 1.5707 1.5707"/>
-            <geometry>
-                <cylinder radius="0.075" length="0.05"/>
-            </geometry>
-        </collision>
-        <inertial>
-            <origin xyz="0 0 0" rpy="0 1.5707 1.5707"/>
-            <mass value="5.0"/>
-            <inertia
-                    ixx="0.1" ixy="0" ixz="0"
-                    iyy="0.1" iyz="0"
-                    izz="0.1"/>
-        </inertial>
-    </link>
-    <joint type="continuous" name="left_wheel_hinge">
+    <link name="front_left_wheel">
+        <visual name="front_left_wheel_visual">
+            <origin xyz="0 0 0" rpy="0 1.5707 1.5707"/>
+            <geometry>
+                <cylinder radius="0.075" length="0.05"/>
+            </geometry>
+        </visual>
+        <collision name="front_left_wheel_collision">
+            <origin xyz="0 0 0" rpy="0 1.5707 1.5707"/>
+            <geometry>
+                <cylinder radius="0.075" length="0.05"/>
+            </geometry>
+        </collision>
+        <inertial>
+            <origin xyz="0 0 0" rpy="0 1.5707 1.5707"/>
+            <mass value="2.5"/>
+            <inertia
+                    ixx="0.1" ixy="0" ixz="0"
+                    iyy="0.1" iyz="0"
+                    izz="0.1"/>
+        </inertial>
+    </link>
+    <link name="back_left_wheel">
+        <visual name="front_left_wheel_visual">
+            <origin xyz="0 0 0" rpy="0 1.5707 1.5707"/>
+            <geometry>
+                <cylinder radius="0.075" length="0.05"/>
+            </geometry>
+        </visual>
+        <collision name="back_left_wheel_collision">
+            <origin xyz="0 0 0" rpy="0 1.5707 1.5707"/>
+            <geometry>
+                <cylinder radius="0.075" length="0.05"/>
+            </geometry>
+        </collision>
+        <inertial>
+            <origin xyz="0 0 0" rpy="0 1.5707 1.5707"/>
+            <mass value="2.5"/>
+            <inertia
+                    ixx="0.1" ixy="0" ixz="0"
+                    iyy="0.1" iyz="0"
+                    izz="0.1"/>
+        </inertial>
+    </link>
+    <link name="front_right_wheel">
+        <visual name="front_right_wheel_visual">
+            <origin xyz="0 0 0" rpy="0 1.5707 1.5707"/>
+            <geometry>
+                <cylinder radius="0.075" length="0.05"/>
+            </geometry>
+        </visual>
+        <collision name="front_right_wheel_collision">
+            <origin xyz="0 0 0" rpy="0 1.5707 1.5707"/>
+            <geometry>
+                <cylinder radius="0.075" length="0.05"/>
+            </geometry>
+        </collision>
+        <inertial>
+            <origin xyz="0 0 0" rpy="0 1.5707 1.5707"/>
+            <mass value="2.5"/>
+            <inertia
+                    ixx="0.1" ixy="0" ixz="0"
+                    iyy="0.1" iyz="0"
+                    izz="0.1"/>
+        </inertial>
+    </link>
+    <link name="back_right_wheel">
+        <visual name="back_right_wheel_visual">
+            <origin xyz="0 0 0" rpy="0 1.5707 1.5707"/>
+            <geometry>
+                <cylinder radius="0.075" length="0.05"/>
+            </geometry>
+        </visual>
+        <collision name="back_right_wheel_collision">
+            <origin xyz="0 0 0" rpy="0 1.5707 1.5707"/>
+            <geometry>
+                <cylinder radius="0.075" length="0.05"/>
+            </geometry>
+        </collision>
+        <inertial>
+            <origin xyz="0 0 0" rpy="0 1.5707 1.5707"/>
+            <mass value="2.5"/>
+            <inertia
+                    ixx="0.1" ixy="0" ixz="0"
+                    iyy="0.1" iyz="0"
+                    izz="0.1"/>
+        </inertial>
+    </link>
+    <joint type="continuous" name="front_left_wheel_hinge">
         <origin xyz="0.1 0.15 -0.025" rpy="0 0 0"/>
-        <child link="left_wheel"/>
-        <parent link="chassis"/>
-        <axis xyz="0 1 0" rpy="0 0 0"/>
-        <limit effort="10000" velocity="1000"/>
-        <dynamics damping="1.0" friction="1.0"/>
-    </joint>
-    <joint type="continuous" name="right_wheel_hinge">
+        <child link="front_left_wheel"/>
+        <parent link="chassis"/>
+        <axis xyz="0 1 0" rpy="0 0 0"/>
+        <limit effort="10000" velocity="1000"/>
+        <dynamics damping="1.0" friction="1.0"/>
+    </joint>
+    <joint type="continuous" name="front_right_wheel_hinge">
         <origin xyz="0.1 -0.15 -0.025" rpy="0 0 0"/>
-        <child link="right_wheel"/>
+        <child link="front_right_wheel"/>
+        <parent link="chassis"/>
+        <axis xyz="0 1 0" rpy="0 0 0"/>
+        <limit effort="10000" velocity="1000"/>
+        <dynamics damping="1.0" friction="1.0"/>
+    </joint>
+    <joint type="continuous" name="back_left_wheel_hinge">
+        <origin xyz="-0.1 0.15 -0.025" rpy="0 0 0"/>
+        <child link="back_left_wheel"/>
+        <parent link="chassis"/>
+        <axis xyz="0 1 0" rpy="0 0 0"/>
+        <limit effort="10000" velocity="1000"/>
+        <dynamics damping="1.0" friction="1.0"/>
+    </joint>
+    <joint type="continuous" name="back_right_wheel_hinge">
+        <origin xyz="-0.1 -0.15 -0.025" rpy="0 0 0"/>
+        <child link="back_right_wheel"/>
         <parent link="chassis"/>
         <axis xyz="0 1 0" rpy="0 0 0"/>
@@ -178,8 +226,8 @@
         <child link="hokuyo"/>
     </joint>
-    <gazebo reference="right_wheel">
+    <gazebo reference="front_right_wheel">
         <material>Gazebo/DarkGrey</material>
     </gazebo>
-    <gazebo reference="left_wheel">
+    <gazebo reference="front_left_wheel">
         <material>Gazebo/DarkGrey</material>
     </gazebo>
